File: hotswap_rgb_oled/dumbpad.kicad_pcb (KiCad board)
At the start: 2 copper layers, 97 x 78.5 mm, 57 parts, among them J1 Conn_01x04_Female

Commit message: Updated silkscreen text
Other:
- board text added: "dumbpad - hotswap - rgb - oled"
Changed lines of the file:
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@@
     (effects (font (size 0.6375 0.6375) (thickness 0.1125)) (justify right))
   )
-  (gr_text "dumbpad - hotswap - rgb" (at 102.2511 143.3786) (layer "F.SilkS")
+  (gr_text "dumbpad - hotswap - rgb - oled" (at 102.2511 143.3786) (layer "F.SilkS")
     (effects (font (size 1.4875 1.4875) (thickness 0.2625)) (justify left bottom))
   )

Commit message: Updated back silkscreen text
Other:
- board text added: "imchipwood x deveth0 x n1ghtBl00d"
- board text removed: "imchipwood x deveth0"
Changed lines of the file:
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@@
     (effects (font (size 0.6375 0.6375) (thickness 0.1125)) (justify right mirror))
   )
-  (gr_text "imchipwood x deveth0" (at 102.2511 143.3786) (layer "B.SilkS")
+  (gr_text "imchipwood x deveth0 x n1ghtBl00d" (at 102.2511 143.3786) (layer "B.SilkS")
     (effects (font (size 1.4875 1.4875) (thickness 0.2625)) (justify right bottom mirror))
   )
